Commit message: Add Lidar into model

File: autorally_description/urdf/autoRallyPlatform.urdf.xacro (robot description, xacro)
@@ -542,4 +542,12 @@
                     wheel_mass="${rear_wheel_mass}"
                     axle_eff_limit="${rear_axle_eff_limit}"/>
+  <property name="M_PI" value="3.14159"/>
+  <xacro:include filename="$(find autorally_description)/urdf/sick_lms1xx_mount.urdf.xacro"/>
+        <sick_lms1xx_mount prefix="base" topic="scan"/>
+      <joint name="laser_mount_joint" type="fixed">
+        <origin xyz="0.0 0 0.2" rpy="0 0 0"/>
+        <parent link="base_link" />
+        <child link="base_laser_mount" />
+      </joint>
   <gazebo>
     <plugin name="gazebo_ros_control" filename="libgazebo_ros_control.so">

File: autorally_description/urdf/autoRallyTrack.urdf (robot description, URDF)
Before this commit: robot track, 1 links, 0 joints
Links:
- link track_link: geometry collision mesh filename=package://autorally_description/urdf/autoRallyTrack.stl scale=0.01 0.01 0.06; visual mesh filename=package://autorally_description/urdf/autoRallyTrack.stl scale=0.01 0.01 0.06

Commit message: Update

File: autorally_description/urdf/autoRallyPlatform.urdf.xacro (robot description, xacro)
@@ -546,5 +546,5 @@
         <sick_lms1xx_mount prefix="base" topic="scan"/>
       <joint name="laser_mount_joint" type="fixed">
-        <origin xyz="0.0 0 0.2" rpy="0 0 0"/>
+        <origin xyz="0.0 0 0.22" rpy="0 0 0"/>
         <parent link="base_link" />
         <child link="base_laser_mount" />
@@ -590,4 +590,12 @@
       <velocityGaussianNoise>0.005 0.005 0.05</velocityGaussianNoise>
     </plugin>
+    <plugin name="robot_groundtruth_sim" filename="libgazebo_ros_p3d.so">
+        <alwaysOn>true</alwaysOn>
+        <updateRate>100.0</updateRate>
+        <bodyName>base_link</bodyName>
+        <topicName>ground_truth/state</topicName>
+        <gaussianNoise>0.0</gaussianNoise>
+        <frameName>map</frameName>
+    </plugin>
     <!-- <plugin name="tire_friction" filename="libTireFrictionPlugin.so">
       <link_name>left_rear_wheel</link_name>

File: autorally_description/urdf/sick_lms1xx.urdf.xacro (robot description, xacro)
@@ -26,5 +26,5 @@
 -->
 <robot xmlns:xacro="http://ros.org/wiki/xacro">
-  <xacro:macro name="sick_lms1xx" params="frame:=laser topic:=scan sample_size:=720 update_rate:=50" >
+  <xacro:macro name="sick_lms1xx" params="frame:=laser topic:=scan sample_size:=70 update_rate:=10" >
     <link name="${frame}">
       <inertial>
@@ -58,7 +58,7 @@
             <horizontal>
               <samples>${sample_size}</samples>
-              <resolution>1</resolution>
-              <min_angle>-2.35619</min_angle>
-              <max_angle>2.35619</max_angle>
+	      <resolution>1</resolution> <!-- 1 -->
+              <min_angle>-1.57</min_angle>  <!-- -2.35619 -->
+              <max_angle>1.57</max_angle>  <!-- 2.35619 -->
             </horizontal>
           </scan>
